File: hardware/laptop thingy/laptop thingy.kicad_sch (KiCad schematic)
At the start: 0 parts

Commit message: fixed file system
Other:
- sheet connectors: file untitled.kicad_sch -> connectors.kicad_sch
Changed lines of the file:
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@@
 			)
 		)
-		(property "Sheetfile" "untitled.kicad_sch"
+		(property "Sheetfile" "connectors.kicad_sch"
 			(at 12.7 160.6046 0)
 			(show_name no)
